File: xds-iso/xds-iso.kicad_sch (KiCad schematic)
At the start: 110 parts, among them J1 USB4085, J2 TGT_JTAG, J3 IF_JTAG, J4 Conn_01x02_Male, SW2 EVQPUD, U1 AP7361EA-33E-13, U2 MSP432E401Y, U3 ISOW7741, U4 ISOW7742, U5 TPD4E004DRYR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

Commit message: Added 5.1k pulldowns to the CC1 and CC2 pins to comply with USB Type C spec
Parts:
- added R34: (no value), Resistor_SMD:R_0402_1005Metric, symbol Device:R_Small_US
- added R35: 5.1k, Resistor_SMD:R_0402_1005Metric, symbol Device:R_Small_US
Connections:
- net GND: now also R34.1, R35.1
- net CC1: now reaches J1.A5 (CC1)
- net CC1: now also R34.2
- net CC2: now reaches J1.B5 (CC2)
- net CC2: now also R35.2
- no-connect marks 82 -> 80
Changed lines of the file:
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@@
     (title "XDS Isolated JTAG/cJTAG/SWD Debugger")
     (date "2022-06-29")
-    (rev "0.2")
+    (rev "0.2b")
     (company "Glasslabs")
   )
@@
   (junction (at 373.38 66.04) (diameter 0) (color 0 0 0 0)
   )
+  (junction (at 71.12 78.74) (diameter 0) (color 0 0 0 0)
+  )
   (junction (at 170.18 48.26) (diameter 0) (color 0 0 0 0)
   )
@@
   (no_connect (at 154.94 190.5))
   (no_connect (at 154.94 193.04))
-  (no_connect (at 55.88 45.72))
-  (no_connect (at 55.88 43.18))
   (no_connect (at 55.88 66.04))
   (no_connect (at 55.88 68.58))
@@
     (stroke (width 0) (type default) (color 0 0 0 0))
   )
+  (wire (pts (xy 76.2 68.58) (xy 78.74 68.58))
+    (stroke (width 0) (type default) (color 0 0 0 0))
+  )
   (wire (pts (xy 314.96 63.5) (xy 314.96 66.04))
     (stroke (width 0) (type default) (color 0 0 0 0))
@@
     (stroke (width 0) (type default) (color 0 0 0 0))
   )
+  (wire (pts (xy 68.58 68.58) (xy 71.12 68.58))
+    (stroke (width 0) (type default) (color 0 0 0 0))
+  )
   (wire (pts (xy 307.34 88.9) (xy 307.34 91.44))
     (stroke (width 0) (type default) (color 0 0 0 0))
@@
     (stroke (width 0) (type default) (color 0 0 0 0))
   )
+  (wire (pts (xy 71.12 81.28) (xy 71.12 78.74))
+    (stroke (width 0) (type default) (color 0 0 0 0))
+  )
   (wire (pts (xy 327.66 160.02) (xy 332.74 160.02))
     (stroke (width 0) (type default) (color 0 0 0 0))
@@
     (stroke (width 0) (type default) (color 0 0 0 0))
   )
+  (wire (pts (xy 71.12 68.58) (xy 71.12 71.12))
+    (stroke (width 0) (type default) (color 0 0 0 0))
+  )
   (wire (pts (xy 205.74 30.48) (xy 205.74 33.02))
     (stroke (width 0) (type default) (color 0 0 0 0))
@@
     (stroke (width 0) (type default) (color 0 0 0 0))
   )
+  (wire (pts (xy 71.12 76.2) (xy 71.12 78.74))
+    (stroke (width 0) (type default) (color 0 0 0 0))
+  )
   (wire (pts (xy 93.98 152.4) (xy 86.36 152.4))
     (stroke (width 0) (type default) (color 0 0 0 0))
@@
     (stroke (width 0) (type default) (color 0 0 0 0))
   )
+  (wire (pts (xy 55.88 45.72) (xy 60.96 45.72))
+    (stroke (width 0) (type default) (color 0 0 0 0))
+  )
   (wire (pts (xy 408.94 96.52) (xy 416.56 96.52))
     (stroke (width 0) (type default) (color 0 0 0 0))
@@
     (stroke (width 0) (type default) (color 0 0 0 0))
   )
+  (wire (pts (xy 55.88 43.18) (xy 60.96 43.18))
+    (stroke (width 0) (type default) (color 0 0 0 0))
+  )
   (wire (pts (xy 236.22 146.05) (xy 236.22 148.59))
     (stroke (width 0) (type default) (color 0 0 0 0))
@@
     (stroke (width 0) (type default) (color 0 0 0 0))
   )
+  (wire (pts (xy 78.74 76.2) (xy 78.74 78.74))
+    (stroke (width 0) (type default) (color 0 0 0 0))
+  )
   (wire (pts (xy 78.74 175.26) (xy 78.74 177.8))
     (stroke (width 0) (type default) (color 0 0 0 0))
@@
     (stroke (width 0) (type default) (color 0 0 0 0))
   )
+  (wire (pts (xy 71.12 78.74) (xy 78.74 78.74))
+    (stroke (width 0) (type default) (color 0 0 0 0))
+  )
   (wire (pts (xy 63.5 162.56) (xy 71.12 162.56))
     (stroke (width 0) (type default) (color 0 0 0 0))
@@
     (stroke (width 0) (type default) (color 0 0 0 0))
   )
+  (wire (pts (xy 78.74 68.58) (xy 78.74 71.12))
+    (stroke (width 0) (type default) (color 0 0 0 0))
+  )
   (wire (pts (xy 187.96 48.26) (xy 187.96 50.8))
     (stroke (width 0) (type default) (color 0 0 0 0))
@@
     (effects (font (size 1.27 1.27)) (justify right bottom))
   )
+  (label "CC1" (at 60.96 43.18 180)
+    (effects (font (size 1.27 1.27)) (justify right bottom))
+  )
   (label "V_{ISOOUT}" (at 313.69 142.24 0)
     (effects (font (size 1.27 1.27)) (justify left bottom))
   )
+  (label "CC2" (at 60.96 45.72 180)
+    (effects (font (size 1.27 1.27)) (justify right bottom))
+  )
   (label "XDS_TMS" (at 321.31 96.52 0)
     (effects (font (size 1.27 1.27)) (justify left bottom))
@@
     (effects (font (size 1.27 1.27)) (justify left bottom))
   )
+  (label "CC2" (at 76.2 68.58 180)
+    (effects (font (size 1.27 1.27)) (justify right bottom))
+  )
   (label "ISO_RX" (at 375.92 93.98 180)
     (effects (font (size 1.27 1.27)) (justify right bottom))
@@
     (effects (font (size 1.27 1.27)) (justify right bottom))
   )
+  (label "CC1" (at 68.58 68.58 180)
+    (effects (font (size 1.27 1.27)) (justify right bottom))
+  )
   (label "USB_DM" (at 144.78 106.68 0)
     (effects (font (size 1.27 1.27)) (justify left bottom))
@@
     (pin "2")
   )
+  (symbol (lib_id "power:GND") (at 71.12 81.28 0) (unit 1)
+    (in_bom yes) (on_board yes) (fields_autoplaced)
+    (property "Reference" "#PWR045" (id 0) (at 71.12 87.63 0)
+      (effects (font (size 1.27 1.27)) hide)
+    )
+    (property "Value" "GND" (id 1) (at 71.12 86.36 0))
+    (property "Footprint" "" (id 2) (at 71.12 81.28 0)
+      (effects (font (size 1.27 1.27)) hide)
+    )
+    (property "Datasheet" "" (id 3) (at 71.12 81.28 0)
+      (effects (font (size 1.27 1.27)) hide)
+    )
+    (pin "1")
+  )
   (symbol (lib_id "power:GND") (at 93.98 165.1 0) (unit 1)
     (in_bom yes) (on_board yes) (fields_autoplaced)
@@
     (pin "2")
   )
+  (symbol (lib_id "Device:R_Small_US") (at 71.12 73.66 180) (unit 1)
+    (in_bom yes) (on_board yes)
+    (property "Reference" "R34" (id 0) (at 66.04 73.66 90))
+    (property "Value" "" (id 1) (at 68.58 73.66 90))
+    (property "Footprint" "Resistor_SMD:R_0402_1005Metric" (id 2) (at 71.12 73.66 0)
+      (effects (font (size 1.27 1.27)) hide)
+    )
+    (property "Datasheet" "~" (id 3) (at 71.12 73.66 0)
+      (effects (font (size 1.27 1.27)) hide)
+    )
+    (pin "1")
+    (pin "2")
+  )
   (symbol (lib_id "Device:C_Small") (at 299.72 93.98 0) (unit 1)
     (in_bom yes) (on_board yes)
@@
     (pin "2")
   )
+  (symbol (lib_id "Device:R_Small_US") (at 78.74 73.66 180) (unit 1)
+    (in_bom yes) (on_board yes)
+    (property "Reference" "R35" (id 0) (at 73.66 73.66 90))
+    (property "Value" "5.1k" (id 1) (at 76.2 73.66 90))
+    (property "Footprint" "Resistor_SMD:R_0402_1005Metric" (id 2) (at 78.74 73.66 0)
+      (effects (font (size 1.27 1.27)) hide)
+    )
+    (property "Datasheet" "~" (id 3) (at 78.74 73.66 0)
+      (effects (font (size 1.27 1.27)) hide)
+    )
+    (pin "1")
+    (pin "2")
+  )
   (symbol (lib_id "Device:C_Small") (at 398.78 30.48 0) (mirror y) (unit 1)
     (in_bom yes) (on_board yes)
@@
       (reference "#PWR044") (unit 1) (value "GND1") (footprint "")
     )
+    (path "/74947056-68ef-4bd4-9974-79f93ba23356"
+      (reference "#PWR045") (unit 1) (value "GND") (footprint "")
+    )
     (path "/2d7f55c2-61f5-44bd-98cc-21201159f319"
       (reference "#PWR0101") (unit 1) (value "GND1") (footprint "")
@@
       (reference "R33") (unit 1) (value "10k") (footprint "Resistor_SMD:R_0402_1005Metric")
     )
+    (path "/92addfab-dbbe-43ac-af64-0d6b00294a7e"
+      (reference "R34") (unit 1) (value "5.1k") (footprint "Resistor_SMD:R_0402_1005Metric")
+    )
+    (path "/99cf65b6-7fd1-4279-ac95-e2f48809fbd6"
+      (reference "R35") (unit 1) (value "5.1k") (footprint "Resistor_SMD:R_0402_1005Metric")
+    )
     (path "/c717d45e-c245-4f0d-8e82-ace6a7adad3d"
